File: som-first-board/SomUSB2.brd (EAGLE design)
At the start: 30.5 x 73.8 mm, 23 parts, among them U1 MP2122

Commit message: SoM First Board v2
Changed value of R8
Parts:
- R8: value 158K -> 150K
Connections:
- net 3V7 renamed 3V8
- net 3V7-REG renamed 3V8-REG
Routing:
- net FB1: track 9.25 -> 6.71 mm
- net 3V8: track 36.1 -> 35.5 mm
Other:
- board text added: "3V8"
- board text added: "SomUSB2 v2"
- board text removed: "3V7"
- board text removed: "SomUSB1 v4"
Changed lines of the file:
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@@
 <?xml version="1.0" encoding="utf-8"?>
 <!DOCTYPE eagle SYSTEM "eagle.dtd">
-<eagle version="9.4.0">
+<eagle version="9.5.2">
 <drawing>
 <settings>
-<setting alwaysvectorfont="yes"/>
+<setting alwaysvectorfont="no"/>
 <setting verticaltext="up"/>
 </settings>
-<grid distance="0.05" unitdist="inch" unit="mm" style="lines" multiple="1" display="no" altdistance="0.025" altunitdist="inch" altunit="mm"/>
+<grid distance="0.05" unitdist="inch" unit="inch" style="lines" multiple="1" display="no" altdistance="0.025" altunitdist="inch" altunit="inch"/>
 <layers>
 <layer number="1" name="Top" color="4" fill="1" visible="yes" active="yes"/>
@@
 <text x="10.16" y="13.335" size="1.27" layer="21" rot="R90">RESET</text>
 <text x="17.145" y="13.335" size="1.27" layer="21" rot="R90">MODE</text>
-<text x="19.05" y="34.29" size="1.27" layer="22" rot="MR0">SomUSB1
-v4</text>
+<text x="19.05" y="34.29" size="1.27" layer="22" rot="MR0">SomUSB2
+v2</text>
 <text x="15.24" y="3.175" size="1.016" layer="21">3V3</text>
-<text x="20.955" y="3.175" size="1.016" layer="21">3V7</text>
+<text x="20.955" y="3.175" size="1.016" layer="21">3V8</text>
 <text x="9.525" y="7.62" size="1.016" layer="21">5V</text>
 <text x="19.685" y="1.27" size="0.6096" layer="21">REG</text>
@@
 <attribute name="VALUE" x="25.4" y="16.637" size="0.4064" layer="51" font="vector"/>
 </element>
-<element name="R8" library="rickk2" package="0603-RES" value="158K" x="25.4" y="15.24" smashed="yes" rot="R180">
-<attribute name="NAME" x="24.765" y="14.478" size="0.4064" layer="51" font="vector" rot="R180"/>
-<attribute name="VALUE" x="26.67" y="14.605" size="0.4064" layer="51" font="vector" rot="R180"/>
-</element>
 <element name="U$3" library="rickk2" package="USB-B-SMT-AMPHENOL" value="USB-MICRO-B-SOCKET-AMPHENOL" x="8.89" y="4.445" smashed="yes"/>
 <element name="S1" library="rickk2" package="SWITCH-MOM-4.5" value="SWITCH-MOM-4.5" x="21.59" y="11.43" smashed="yes" rot="R90">
@@
 <element name="JP1" library="rickk2" package="1X02" value="M02PTH" x="5.08" y="8.255" smashed="yes"/>
 <element name="U$1" library="rickk2" package="M2-STANDOFF" value="M2-STANDOFF" x="15.24" y="69.94" smashed="yes"/>
+<element name="R8" library="rickk2" package="0603-RES" value="150K" x="25.4" y="15.24" smashed="yes" rot="R180">
+<attribute name="NAME" x="26.289" y="14.478" size="0.4064" layer="51" font="vector" rot="R180"/>
+<attribute name="VALUE" x="26.416" y="16.383" size="0.4064" layer="51" font="vector" rot="R180"/>
+</element>
 </elements>
 <signals>
@@
 <via x="4.445" y="16.51" extent="1-16" drill="0.35"/>
 <contactref element="U1" pad="5"/>
-<contactref element="R8" pad="1"/>
 <contactref element="R6" pad="1"/>
 <contactref element="C2" pad="2"/>
@@
 <contactref element="S1" pad="2"/>
 <contactref element="S2" pad="2"/>
+<contactref element="R8" pad="1"/>
 </signal>
 <signal name="/MODE">
@@
 <signal name="FB1">
 <contactref element="U1" pad="8"/>
-<contactref element="R8" pad="2"/>
 <contactref element="R7" pad="1"/>
-<wire x1="24.55" y1="17.78" x2="24.55" y2="15.24" width="0.254" layer="1"/>
 <wire x1="23.2506" y1="11.07426875" x2="23.2506" y2="13.05573125" width="0.254" layer="1"/>
-<wire x1="24.55" y1="15.24" x2="24.55" y2="14.35513125" width="0.254" layer="1"/>
-<wire x1="24.55" y1="14.35513125" x2="23.2506" y2="13.05573125" width="0.254" layer="1"/>
+<wire x1="24.55" y1="14.35513125" x2="24.147434375" y2="13.952565625" width="0.254" layer="1"/>
+<wire x1="24.147434375" y1="13.952565625" x2="23.2506" y2="13.05573125" width="0.254" layer="1"/>
 <wire x1="24.425" y1="9.555" x2="24.425" y2="9.89986875" width="0.254" layer="1"/>
 <wire x1="24.425" y1="9.89986875" x2="23.2506" y2="11.07426875" width="0.254" layer="1"/>
-</signal>
-<signal name="3V7">
-<wire x1="26.525" y1="32.53" x2="27.305" y2="31.75" width="0.254" layer="1"/>
-<contactref element="J1" pad="2"/>
-<contactref element="J1" pad="4"/>
-<contactref element="J1" pad="6"/>
-<contactref element="J1" pad="8"/>
-<wire x1="26.525" y1="32.53" x2="24.61" y2="32.53" width="0.254" layer="1"/>
-<wire x1="24.61" y1="32.53" x2="24.11" y2="32.53" width="0.254" layer="1"/>
-<wire x1="24.11" y1="32.53" x2="23.61" y2="32.53" width="0.254" layer="1"/>
-<wire x1="23.61" y1="32.53" x2="23.11" y2="32.53" width="0.254" layer="1"/>
-<contactref element="SJ2" pad="2"/>
-<via x="26.67" y="22.225" extent="1-16" drill="0.35"/>
-<wire x1="27.305" y1="22.86" x2="26.67" y2="22.225" width="0.254" layer="1"/>
-<wire x1="27.305" y1="31.75" x2="27.305" y2="22.86" width="0.254" layer="1"/>
-<wire x1="26.2664" y1="8.6543875" x2="26.2664" y2="8.1096125" width="0.254" layer="16"/>
-<wire x1="26.67" y1="22.225" x2="26.67" y2="9.0579875" width="0.254" layer="16"/>
-<wire x1="26.67" y1="7.7060125" x2="26.67" y2="3.175" width="0.254" layer="16"/>
-<wire x1="26.67" y1="9.0579875" x2="26.2664" y2="8.6543875" width="0.254" layer="16"/>
-<wire x1="26.2664" y1="8.1096125" x2="26.67" y2="7.7060125" width="0.254" layer="16"/>
-<wire x1="26.67" y1="3.175" x2="25.4" y2="1.905" width="0.254" layer="16"/>
-<wire x1="25.4" y1="1.905" x2="24.765" y2="1.905" width="0.254" layer="16"/>
+<contactref element="R8" pad="2"/>
+<wire x1="24.55" y1="15.24" x2="24.55" y2="14.35513125" width="0.254" layer="1"/>
+<wire x1="24.55" y1="15.24" x2="24.55" y2="17.78" width="0" layer="19" extent="1-1"/>
 </signal>
 <signal name="VUSB">
@@
 <wire x1="24.13" y1="4.445" x2="18.68" y2="4.445" width="0.254" layer="1"/>
 </signal>
-<signal name="3V7-REG">
+<signal name="3V8-REG">
 <contactref element="R7" pad="2"/>
 <contactref element="L2" pad="2"/>
@@
 <wire x1="25.4" y1="22.225" x2="25.4" y2="3.81" width="0.254" layer="16"/>
 </signal>
+<signal name="3V8">
+<contactref element="SJ2" pad="2"/>
+<wire x1="26.525" y1="32.53" x2="27.305" y2="31.75" width="0.254" layer="1"/>
+<contactref element="J1" pad="2"/>
+<contactref element="J1" pad="4"/>
+<contactref element="J1" pad="6"/>
+<contactref element="J1" pad="8"/>
+<wire x1="26.525" y1="32.53" x2="24.61" y2="32.53" width="0.254" layer="1"/>
+<wire x1="24.61" y1="32.53" x2="24.11" y2="32.53" width="0.254" layer="1"/>
+<wire x1="24.11" y1="32.53" x2="23.61" y2="32.53" width="0.254" layer="1"/>
+<wire x1="23.61" y1="32.53" x2="23.11" y2="32.53" width="0.254" layer="1"/>
+<via x="26.67" y="22.225" extent="1-16" drill="0.35"/>
+<wire x1="27.305" y1="22.86" x2="26.67" y2="22.225" width="0.254" layer="1"/>
+<wire x1="27.305" y1="31.75" x2="27.305" y2="22.86" width="0.254" layer="1"/>
+<wire x1="26.2664" y1="8.6543875" x2="26.2664" y2="8.1096125" width="0.254" layer="16"/>
+<wire x1="26.67" y1="22.225" x2="26.67" y2="9.0579875" width="0.254" layer="16"/>
+<wire x1="26.67" y1="7.7060125" x2="26.67" y2="3.175" width="0.254" layer="16"/>
+<wire x1="26.67" y1="9.0579875" x2="26.2664" y2="8.6543875" width="0.254" layer="16"/>
+<wire x1="26.2664" y1="8.1096125" x2="26.67" y2="7.7060125" width="0.254" layer="16"/>
+<wire x1="26.67" y1="3.175" x2="25.4" y2="1.905" width="0.254" layer="16"/>
+<wire x1="24.765" y1="1.905" x2="25.4" y2="1.905" width="0" layer="19" extent="16-16"/>
+</signal>
 </signals>

Commit message: v3
- Swap pins D2 and D3
Parts:
- J1: value (none) -> SPARK_M.2EKEY
Other:
- board text added: "SomUSB2 v3"
- board text removed: "SomUSB2 v2"
Changed lines of the file:
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@@
 <?xml version="1.0" encoding="utf-8"?>
 <!DOCTYPE eagle SYSTEM "eagle.dtd">
-<eagle version="9.5.2">
+<eagle version="9.6.2">
 <drawing>
 <settings>
@@
 <layer number="1" name="Top" color="4" fill="1" visible="yes" active="yes"/>
 <layer number="2" name="Route2" color="16" fill="1" visible="no" active="no"/>
+<layer number="3" name="Route3" color="17" fill="1" visible="no" active="no"/>
+<layer number="4" name="Route4" color="18" fill="1" visible="no" active="no"/>
+<layer number="5" name="Route5" color="19" fill="1" visible="no" active="no"/>
+<layer number="6" name="Route6" color="25" fill="1" visible="no" active="no"/>
+<layer number="7" name="Route7" color="26" fill="1" visible="no" active="no"/>
+<layer number="8" name="Route8" color="27" fill="1" visible="no" active="no"/>
+<layer number="9" name="Route9" color="28" fill="1" visible="no" active="no"/>
+<layer number="10" name="Route10" color="29" fill="1" visible="no" active="no"/>
+<layer number="11" name="Route11" color="30" fill="1" visible="no" active="no"/>
+<layer number="12" name="Route12" color="20" fill="1" visible="no" active="no"/>
+<layer number="13" name="Route13" color="21" fill="1" visible="no" active="no"/>
+<layer number="14" name="Route14" color="22" fill="1" visible="no" active="no"/>
 <layer number="15" name="Route15" color="23" fill="1" visible="no" active="no"/>
 <layer number="16" name="Bottom" color="1" fill="1" visible="yes" active="yes"/>
@@
 <text x="17.145" y="13.335" size="1.27" layer="21" rot="R90">MODE</text>
 <text x="19.05" y="34.29" size="1.27" layer="22" rot="MR0">SomUSB2
-v2</text>
+v3</text>
 <text x="15.24" y="3.175" size="1.016" layer="21">3V3</text>
 <text x="20.955" y="3.175" size="1.016" layer="21">3V8</text>
@@
 <attribute name="NAME" x="4.6228" y="12.7254" size="0.6096" layer="48" rot="R90"/>
 </element>
-<element name="J1" library="rickk2" package="SPARK_M.2EKEY-LESS-CREAM" value="" x="15.24" y="27.94" smashed="yes" rot="R180">
+<element name="J1" library="rickk2" package="SPARK_M.2EKEY-LESS-CREAM" value="SPARK_M.2EKEY" x="15.24" y="27.94" smashed="yes" rot="R180">
 <attribute name="VALUE" x="15.0512" y="21.8332" size="1.27" layer="51" rot="R180"/>
 </element>
