File: som-first-board/SomUSB2.sch (EAGLE design)
At the start: 23 parts, among them J1 SPARK_M.2EKEY, U1 MP2122

Commit message: SoM First Board v2
Changed value of R8
Parts:
- R8: value 158K -> 150K; device rickk2:RES-158K-0603 -> rickk2:RES-150K-0603
Connections:
- net 3V7 renamed 3V8
- net 3V7-REG renamed 3V8-REG

Commit message: v3
- Swap pins D2 and D3
Changed lines of the file:
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@@
 <?xml version="1.0" encoding="utf-8"?>
 <!DOCTYPE eagle SYSTEM "eagle.dtd">
-<eagle version="9.5.2">
+<eagle version="9.6.2">
 <drawing>
 <settings>
@@
 <layer number="1" name="Top" color="4" fill="1" visible="no" active="no"/>
 <layer number="2" name="Route2" color="1" fill="3" visible="no" active="no"/>
+<layer number="3" name="Route3" color="17" fill="1" visible="no" active="no"/>
+<layer number="4" name="Route4" color="18" fill="1" visible="no" active="no"/>
+<layer number="5" name="Route5" color="19" fill="1" visible="no" active="no"/>
+<layer number="6" name="Route6" color="25" fill="1" visible="no" active="no"/>
+<layer number="7" name="Route7" color="26" fill="1" visible="no" active="no"/>
+<layer number="8" name="Route8" color="27" fill="1" visible="no" active="no"/>
+<layer number="9" name="Route9" color="28" fill="1" visible="no" active="no"/>
+<layer number="10" name="Route10" color="29" fill="1" visible="no" active="no"/>
+<layer number="11" name="Route11" color="30" fill="1" visible="no" active="no"/>
+<layer number="12" name="Route12" color="20" fill="1" visible="no" active="no"/>
+<layer number="13" name="Route13" color="21" fill="1" visible="no" active="no"/>
+<layer number="14" name="Route14" color="22" fill="1" visible="no" active="no"/>
 <layer number="15" name="Route15" color="4" fill="6" visible="no" active="no"/>
 <layer number="16" name="Bottom" color="1" fill="1" visible="no" active="no"/>
@@
 <part name="S1" library="rickk2" deviceset="SWITCH-MOM-4.5" device=""/>
 <part name="S2" library="rickk2" deviceset="SWITCH-MOM-4.5" device=""/>
-<part name="J1" library="rickk2" deviceset="SPARK_M.2EKEY" device="" value=""/>
+<part name="J1" library="rickk2" deviceset="SPARK_M.2EKEY" device="" value="SPARK_M.2EKEY"/>
 <part name="SJ1" library="rickk2" deviceset="JUMPER-PTH-2-NO" device=""/>
 <part name="SJ2" library="rickk2" deviceset="JUMPER-PTH-2-NO" device=""/>
